Commit message: launch arguments

File: miniarm_ros/miniarm_description/urdf/miniarm.urdf (robot description, URDF)
Before this commit: robot miniarm, 18 links, 17 joints
Joints:
- joint miniarm_joint3: limit lower=-1.5708 upper=2.356195 effort=10 velocity=2 -> lower=-0.785 upper=2.3561 effort=10 velocity=2; origin xyz=0.0 0.12 0 rpy=0 3.141592653589793 0 -> xyz=0.0 0.12 0 rpy=0 3.1416 1.5708
