Commit message: Checkpoint bounded arm controls, gripper camera firmware, and repaired ROS model

File: ros2/miniarm_description/urdf/miniarm.urdf (robot description, URDF)
Before this commit: robot miniarm, 18 links, 17 joints
Links:
- link miniarm_base: geometry collision mesh filename=package://miniarm_description/meshes/Base.STL scale=0.001 0.001 0.001; visual mesh filename=package://miniarm_description/meshes/Base.STL scale=0.001 0.001 0.001
- link miniarm_electronics: geometry collision mesh filename=package://miniarm_description/meshes/electronics_deck.STL scale=0.001 0.001 0.001; visual mesh filename=package://miniarm_description/meshes/electronics_deck.STL scale=0.001 0.001 0.001
- link miniarm_gripper_link: geometry collision mesh filename=package://miniarm_description/meshes/link_6.STL scale=0.001 0.001 0.001; visual mesh filename=package://miniarm_description/meshes/link_6.STL scale=0.001 0.001 0.001
- link miniarm_left_bottom_knuckle_link: geometry collision mesh filename=package://miniarm_description/meshes/gripper_link.STL scale=0.001 0.001 0.001; visual mesh filename=package://miniarm_description/meshes/gripper_link.STL scale=0.001 0.001 0.001
- link miniarm_left_finger_link: geometry collision mesh filename=package://miniarm_description/meshes/gripper_finger.STL scale=0.001 0.001 0.001; visual mesh filename=package://miniarm_description/meshes/gripper_finger.STL scale=0.001 0.001 0.001
- link miniarm_left_inner_bottom_knuckle_link: geometry collision mesh filename=package://miniarm_description/meshes/gripper_link.STL scale=0.001 0.001 0.001; visual mesh filename=package://miniarm_description/meshes/gripper_link.STL scale=0.001 0.001 0.001
- link miniarm_left_inner_knuckle_link: geometry collision mesh filename=package://miniarm_description/meshes/gripper_link.STL scale=0.001 0.001 0.001; visual mesh filename=package://miniarm_description/meshes/gripper_link.STL scale=0.001 0.001 0.001
- link miniarm_left_knuckle_link: geometry collision mesh filename=package://miniarm_description/meshes/gripper_link.STL scale=0.001 0.001 0.001; visual mesh filename=package://miniarm_description/meshes/gripper_link.STL scale=0.001 0.001 0.001
- link miniarm_link1: geometry collision mesh filename=package://miniarm_description/meshes/link_1.STL scale=0.001 0.001 0.001; visual mesh filename=package://miniarm_description/meshes/link_1.STL scale=0.001 0.001 0.001
- link miniarm_link2: geometry collision mesh filename=package://miniarm_description/meshes/link_2.STL scale=0.001 0.001 0.001; visual mesh filename=package://miniarm_description/meshes/link_2.STL scale=0.001 0.001 0.001
- link miniarm_link3: geometry collision mesh filename=package://miniarm_description/meshes/link_3.STL scale=0.001 0.001 0.001; visual mesh filename=package://miniarm_description/meshes/link_3.STL scale=0.001 0.001 0.001
- link miniarm_link4: geometry collision mesh filename=package://miniarm_description/meshes/link_4.STL scale=0.001 0.001 0.001; visual mesh filename=package://miniarm_description/meshes/link_4.STL scale=0.001 0.001 0.001
- link miniarm_link5: geometry collision mesh filename=package://miniarm_description/meshes/link_5.STL scale=0.001 0.001 0.001; visual mesh filename=package://miniarm_description/meshes/link_5.STL scale=0.001 0.001 0.001
- link miniarm_right_bottom_knuckle_link: geometry collision mesh filename=package://miniarm_description/meshes/gripper_link.STL scale=0.001 0.001 0.001; visual mesh filename=package://miniarm_description/meshes/gripper_link.STL scale=0.001 0.001 0.001
- link miniarm_right_finger_link: geometry collision mesh filename=package://miniarm_description/meshes/gripper_finger.STL scale=0.001 0.001 0.001; visual mesh filename=package://miniarm_description/meshes/gripper_finger.STL scale=0.001 0.001 0.001
- link miniarm_right_inner_bottom_knuckle_link: geometry collision mesh filename=package://miniarm_description/meshes/gripper_link.STL scale=0.001 0.001 0.001; visual mesh filename=package://miniarm_description/meshes/gripper_link.STL scale=0.001 0.001 0.001
- link miniarm_right_inner_knuckle_link: geometry collision mesh filename=package://miniarm_description/meshes/gripper_link.STL scale=0.001 0.001 0.001; visual mesh filename=package://miniarm_description/meshes/gripper_link.STL scale=0.001 0.001 0.001
- link miniarm_right_knuckle_link: geometry collision mesh filename=package://miniarm_description/meshes/gripper_link.STL scale=0.001 0.001 0.001; visual mesh filename=package://miniarm_description/meshes/gripper_link.STL scale=0.001 0.001 0.001

File: ros2/miniarm_moveit_config/config/miniarm.ros2_control.xacro (robot description, xacro)
@@ -1,47 +1,26 @@
 <?xml version="1.0"?>
 <robot xmlns:xacro="http://www.ros.org/wiki/xacro">
-    <xacro:macro name="miniarm_ros2_control" params="name initial_positions_file">
-        <xacro:property name="initial_positions" value="${load_yaml(initial_positions_file)['initial_positions']}"/>
-        <ros2_control name="${name}" type="system">
-            <hardware>
-                <plugin>fake_components/GenericSystem</plugin>
-            </hardware>
-            <joint name="miniarm_joint1">
-                <param name="initial_position">${initial_positions['miniarm_joint1']}</param>
-                <command_interface name="position" />
-                <state_interface name="position"/>
-                <state_interface name="velocity"/>
-            </joint>
-            <joint name="miniarm_joint2">
-                <param name="initial_position">${initial_positions['miniarm_joint2']}</param>
-                <command_interface name="position" />
-                <state_interface name="position"/>
-                <state_interface name="velocity"/>
-            </joint>
-            <joint name="miniarm_joint3">
-                <param name="initial_position">${initial_positions['miniarm_joint3']}</param>
-                <command_interface name="position" />
-                <state_interface name="position"/>
-                <state_interface name="velocity"/>
-            </joint>
-            <joint name="miniarm_joint4">
-                <param name="initial_position">${initial_positions['miniarm_joint4']}</param>
-                <command_interface name="position" />
-                <state_interface name="position"/>
-                <state_interface name="velocity"/>
-            </joint>
-            <joint name="miniarm_joint5">
-                <param name="initial_position">${initial_positions['miniarm_joint5']}</param>
-                <command_interface name="position" />
-                <state_interface name="position"/>
-                <state_interface name="velocity"/>
-            </joint>
-            <joint name="miniarm_joint6">
-                <param name="initial_position">${initial_positions['miniarm_joint6']}</param>
-                <command_interface name="position" />
-                <state_interface name="position"/>
-                <state_interface name="velocity"/>
-            </joint>
-        </ros2_control>
-    </xacro:macro>
+  <xacro:macro name="miniarm_mock_joint" params="joint_name initial_positions">
+    <joint name="${joint_name}">
+      <command_interface name="position"/>
+      <state_interface name="position">
+        <param name="initial_value">${initial_positions[joint_name]}</param>
+      </state_interface>
+      <state_interface name="velocity"/>
+    </joint>
+  </xacro:macro>
+  <xacro:macro name="miniarm_ros2_control" params="name initial_positions_file">
+    <xacro:property name="initial_positions" value="${xacro.load_yaml(initial_positions_file)['initial_positions']}"/>
+    <!-- Intentionally no serial/network plugin or hardware-selection argument. -->
+    <ros2_control name="${name}" type="system">
+      <hardware><plugin>mock_components/GenericSystem</plugin></hardware>
+      <xacro:miniarm_mock_joint joint_name="miniarm_joint1" initial_positions="${initial_positions}"/>
+      <xacro:miniarm_mock_joint joint_name="miniarm_joint2" initial_positions="${initial_positions}"/>
+      <xacro:miniarm_mock_joint joint_name="miniarm_joint3" initial_positions="${initial_positions}"/>
+      <xacro:miniarm_mock_joint joint_name="miniarm_joint4" initial_positions="${initial_positions}"/>
+      <xacro:miniarm_mock_joint joint_name="miniarm_joint5" initial_positions="${initial_positions}"/>
+      <xacro:miniarm_mock_joint joint_name="miniarm_gripper_link_joint" initial_positions="${initial_positions}"/>
+      <xacro:miniarm_mock_joint joint_name="miniarm_gripper_joint" initial_positions="${initial_positions}"/>
+    </ros2_control>
+  </xacro:macro>
 </robot>

File: ros2/miniarm_moveit_config/config/miniarm.urdf.xacro (robot description, xacro)
@@ -1,5 +1,5 @@
 <?xml version="1.0"?>
 <robot xmlns:xacro="http://www.ros.org/wiki/xacro" name="miniarm">
-    <xacro:arg name="initial_positions_file" default="initial_positions.yaml" />
+    <xacro:arg name="initial_positions_file" default="$(find miniarm_moveit_config)/config/initial_positions.yaml" />
     <!-- Import miniarm urdf file -->
     <xacro:include filename="$(find miniarm_description)/urdf/miniarm.urdf" />
@@ -7,5 +7,5 @@
     <xacro:include filename="miniarm.ros2_control.xacro" />
     <!-- <xacro:include filename="miniarm_hand.ros2_control.xacro" /> -->
-    <xacro:miniarm_ros2_control name="MiniarmFakeSystem" initial_positions_file="$(arg initial_positions_file)"/>
+    <xacro:miniarm_ros2_control name="MiniarmMockSystem" initial_positions_file="$(arg initial_positions_file)"/>
     <!-- <xacro:miniarm_hand_ros2_control name="PandaHandFakeSystem"/> -->
 </robot>
